File: pcb/tool_checkout_cabinet/tool_checkout_cabinet_modules.kicad_pcb (KiCad board)
At the start: 2 copper layers, 9 parts, among them J1 Barrel_Jack, Q2 AOD4184A, U1 ESP32-DEVKITC-32D

Commit message: v1 update
Parts:
- removed B1: SPARKFUN_LOGIC_LEVEL_CONVERTER, SPARKFUN_LOGIC_LEVEL_CONVERTER
- removed L1: JST_EH_B2B-EH-A_1x02_P2.50mm_Vertical, Connector_JST:JST_EH_B2B-EH-A_1x02_P2.50mm_Vertical
- removed the REF** at (139.7, 125.7)
- removed the REF** at (106.7, 16.5)
- added J1-ALT: PinHeader_1x02_P2.54mm_Vertical, Connector_PinHeader_2.54mm:PinHeader_1x02_P2.54mm_Vertical, F.Cu at (201.2, 107.2)
- added J2: Screw_Terminal_01x04, TerminalBlock:TerminalBlock_bornier-4_P5.08mm, F.Cu at (195.1, 141.7)
- added J3: Conn_01x20_Male, Connector_PinHeader_2.54mm:PinHeader_1x20_P2.54mm_Vertical, F.Cu at (169.2, 55.9)
- added J4: Conn_01x20_Male, Connector_PinHeader_2.54mm:PinHeader_1x20_P2.54mm_Vertical, F.Cu at (207.5, 104.1)
- added J5: Screw_Terminal_01x02, TerminalBlock:TerminalBlock_bornier-2_P5.08mm, F.Cu at (168.1, 122.4)
- added J5-ALT: PinHeader_1x02_P2.54mm_Vertical, Connector_PinHeader_2.54mm:PinHeader_1x02_P2.54mm_Vertical, F.Cu at (168.1, 129.0)
- added J6: Screw_Terminal_01x02, TerminalBlock:TerminalBlock_bornier-2_P5.08mm, F.Cu at (206.8, 129.0)
- added J6-ALT: PinHeader_1x02_P2.54mm_Vertical, Connector_PinHeader_2.54mm:PinHeader_1x02_P2.54mm_Vertical, F.Cu at (212.6, 130.0)
- added Q1: DMG2302U, Package_TO_SOT_SMD:SOT-23, F.Cu at (190.0, 132.0)
- added R1: 10k, Resistor_SMD:R_0603_1608Metric_Pad1.05x0.95mm_HandSolder, F.Cu at (176.0, 128.5)
- added R2: 4k7, Resistor_SMD:R_0603_1608Metric_Pad1.05x0.95mm_HandSolder, F.Cu at (176.0, 132.6)
- added R3: 10k, Resistor_SMD:R_0603_1608Metric_Pad1.05x0.95mm_HandSolder, F.Cu at (182.5, 128.3)
- added R4: 4k7, Resistor_SMD:R_0603_1608Metric_Pad1.05x0.95mm_HandSolder, F.Cu at (182.4, 132.5)
- added REF**: MountingHole_3.2mm_M3, MountingHole:MountingHole_3.2mm_M3, F.Cu at (211.7, 51.6)
- added REF**: MountingHole_3.2mm_M3, MountingHole:MountingHole_3.2mm_M3, F.Cu at (163.8, 51.6)
- added REF**: MountingHole_3.2mm_M3, MountingHole:MountingHole_3.2mm_M3, F.Cu at (207.0, 143.0)
- added REF**: MountingHole_3.2mm_M3, MountingHole:MountingHole_3.2mm_M3, F.Cu at (169.2, 141.5)
- D1: value MRA4004T3G -> V8PAM10S-M3_H; footprint Diode_SMD:D_SMA -> SamacSys_Parts:V8PAM10SHM3H
- J1: value Barrel_Jack -> Screw_Terminal_01x02; footprint Connector_BarrelJack:BarrelJack_CUI_PJ-102AH_Horizontal -> TerminalBlock:TerminalBlock_bornier-2_P5.08mm
- Q2: footprint DPAK228P994X240-4N -> AOD4184A:DPAK228P994X240-4N
- U1: value ESP32-DEVKITC-32D -> ESP32_DevKit_V1_DOIT; footprint MODULE_ESP32-DEVKITC-32D -> esp32_devkit_v1_doit:esp32_devkit_v1_doit
- moved J1 93.8 mm to (206.8, 114.8)
- moved Q2 92.1 mm to (194.1, 125.0), turned to 270 degrees
- moved D1 89.3 mm to (198.6, 132.6), turned to 270 degrees
- moved U1 72.5 mm to (188.2, 55.8)
- moved A1 56.2 mm to (190.8, 115.1)
Connections:
- A1 pad 1: +12V -> J6-12v
- A1 pad 3: Net-(A1-Pad3) -> +5V
- A1 pad 4: Net-(A1-Pad4) -> GND
- D1 pad 1: Net-(A1-Pad4) -> J6-12v
- J1 pad 1: +12V -> GND
- J1 pad 2: GND -> J6-12v
- Q2 pad 1: Net-(Q2-Pad1) -> IO4
- Q2 pad 3: Net-(A1-Pad4) -> GND
- U1 pad 14: Net-(A1-Pad4) -> GND
- U1 pad 15: Net-(U1-Pad15) -> +5V
- U1 pad 17: Net-(U1-Pad17) -> GND
- U1 pad 19: Net-(A1-Pad3) -> Net-(J4-Pad9)
- U1 pad 20: Net-(A1-Pad4) -> IO4
- U1 pad 26: Net-(A1-Pad4) -> Net-(J4-Pad16)
- U1 pad 4: Net-(U1-Pad4) -> IO34
- U1 pad 5: Net-(B1-PadLV2) -> IO35
- U1 pad 6: Net-(B1-PadLV1) -> IO32
Routing:
- net Net-(A1-Pad4): track 118.1 -> 0.00 mm
- net Net-(A1-Pad3): track 99.9 -> 0.00 mm
- net IO34: track 0.00 -> 84.0 mm
- net IO32: track 0.00 -> 80.6 mm
- net IO35: track 0.00 -> 80.6 mm
- net IO4: track 0.00 -> 71.5 mm
- net J6-12v: track 0.00 -> 70.6 mm
- net Net-(Q2-Pad1): track 64.1 -> 0.00 mm
- net Net-(D1-Pad2): track 9.07 -> 52.3 mm, vias 0 -> 4
- net GND: track 143.1 -> 109.6 mm, vias 0 -> 7
- net Net-(B1-PadLV1): track 33.3 -> 0.00 mm
- net +12V: track 29.2 -> 0.00 mm
- net Net-(B1-PadLV2): track 29.0 -> 0.00 mm
- net (no net): track 25.4 -> 0.00 mm
- net +5V: track 0.00 -> 20.9 mm
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- added copper zone on B.Cu, net GND
Other:
- board outline added: 54.9 x 99.3 mm
- net class +12v added: clearance 0.55, trace_width 1.8, via_dia 0.8, via_drill 0.4
- net class Default: clearance 0.2 -> 0.55
- rule trace_clearance: 0.2 -> 0.55
- board text added: "12v"
- board text added: "12v INPUT"
- board text added: "D0"
- board text added: "D1"
- board text added: "DOOR SWITCH"
- board text added: "Evan@EvanLott.com"
- board text added: "GND"
- board text added: "LOCK"
- board text added: "RFID READER"
- board text added: "RFID WIFI Lock V1 Jan. 2021"
