File: pcb/tool_checkout_cabinet/tool_checkout_cabinet_modules.sch (KiCad schematic (older format))
At the start: 7 parts, among them J1 Barrel_Jack, Q2 AOD4184A, U1 ESP32-DEVKITC-32D

Commit message: v1 update
Parts:
- removed B1: SPARKFUN_LOGIC_LEVEL_CONVERTER, SPARKFUN_LOGIC_LEVEL_CONVERTER, symbol SparkFun-Boards:SPARKFUN_LOGIC_LEVEL_CONVERTER
- removed D1: MRA4004T3G, Diode_SMD:D_SMA, symbol Diode:MRA4004T3G
- removed J1: Barrel_Jack, Connector_BarrelJack:BarrelJack_CUI_PJ-102AH_Horizontal, symbol Connector:Barrel_Jack
- removed U1: ESP32-DEVKITC-32D, MODULE_ESP32-DEVKITC-32D, symbol ESP32-DEVKITC-32D:ESP32-DEVKITC-32D
- added D1: V8PAM10S-M3_H, SamacSys_Parts:V8PAM10SHM3H, symbol SamacSys_Parts:V8PAM10S-M3_H
- added J1, J5, J6: Screw_Terminal_01x02, TerminalBlock:TerminalBlock_bornier-2_P5.08mm, symbol Connector:Screw_Terminal_01x02
- added J2: Screw_Terminal_01x04, TerminalBlock:TerminalBlock_bornier-4_P5.08mm, symbol Connector:Screw_Terminal_01x04
- added J3, J4: Conn_01x20_Male, Connector_PinHeader_2.54mm:PinHeader_1x20_P2.54mm_Vertical, symbol Connector:Conn_01x20_Male
- added Q1: DMG2302U, Package_TO_SOT_SMD:SOT-23, symbol Transistor_FET:DMG2302U
- added R1, R3: 10k, Resistor_SMD:R_0603_1608Metric_Pad1.05x0.95mm_HandSolder, symbol Device:R_US
- added R2, R4: 4k7, Resistor_SMD:R_0603_1608Metric_Pad1.05x0.95mm_HandSolder, symbol Device:R_US
- added U1: ESP32_DevKit_V1_DOIT, esp32_devkit_v1_doit:esp32_devkit_v1_doit, symbol esp32_devkit_v1_doit:ESP32_DevKit_V1_DOIT
- L1: footprint Connector_JST:JST_EH_B2B-EH-A_1x02_P2.50mm_Vertical -> (none)
- Q2: footprint DPAK228P994X240-4N -> AOD4184A:DPAK228P994X240-4N
Connections:
- net +12V: now also L1.1, D1.1, J1.2 (Pin_2), J2.1 (Pin_1), J6.1 (Pin_1)
- net GND: now also A1.4 (OUT-), Q2.3, J1.1 (Pin_1), J2.2 (Pin_2), J3.14 (Pin_14), J4.7 (Pin_7), J5.2 (Pin_2), Q1.2 (S), R1.1, R3.1, U1.14 (GND), U1.17 (GND)
- net +5V: now reaches A1.3 (OUT+)
- net +5V: now also J3.15 (Pin_15), U1.15 (VIN)
- net IO4: now reaches Q2.1
- net IO4: now also J4.10 (Pin_10), Q1.1 (G), U1.20 (IO4)
- net J6-GND: now reaches Q2.4
- net J6-GND: now also L1.2, D1.2, J6.2 (Pin_2), Q1.3 (D); no longer L1.1
- new net: J3.1 (Pin_1), U1.1 (EN)
- new net: J3.10 (Pin_10), U1.10 (IO27)
- new net: J3.11 (Pin_11), U1.11 (IO14)
- new net: J3.12 (Pin_12), U1.12 (IO12)
- new net: J3.13 (Pin_13), U1.13 (IO13)
- new net: J3.2 (Pin_2), U1.2 (SENSOR_VP)
- new net: J3.3 (Pin_3), U1.3 (SENSOR_VN)
- new net: J3.7 (Pin_7), U1.7 (IO33)
- new net: J3.8 (Pin_8), U1.8 (IO25)
- new net: J3.9 (Pin_9), U1.9 (IO26)
- new net: J4.11 (Pin_11), U1.21 (RX2/IO16)
- new net: J4.12 (Pin_12), U1.22 (TX2/IO17)
- new net: J4.13 (Pin_13), U1.23 (IO5)
- new net: J4.14 (Pin_14), U1.24 (IO18)
- new net: J4.15 (Pin_15), U1.25 (IO19)
- new net: J4.16 (Pin_16), U1.26 (IO21)
- new net: J4.17 (Pin_17), U1.27 (RXD0/IO3)
- new net: J4.18 (Pin_18), U1.28 (TXD0/IO1)
- new net: J4.19 (Pin_19), U1.29 (IO22)
- new net: J4.20 (Pin_20), U1.30 (IO23)
- new net: J4.6 (Pin_6), U1.16 (3V3)
- new net: J4.8 (Pin_8), U1.18 (IO15)
- new net: J4.9 (Pin_9), U1.19 (IO2)
- new net: J2.3 (Pin_3), R4.2
- new net: J2.4 (Pin_4), R2.2
- new net IO32: J3.6 (Pin_6), J5.1 (Pin_1), U1.6 (IO32)
- new net IO34: J3.4 (Pin_4), R3.2, R4.1, U1.4 (IO34)
- new net IO35: J3.5 (Pin_5), R1.2, R2.1, U1.5 (IO35)
- no-connect marks 0 -> 10
Other:
- note added: "Alternate Transistor Footprint (TO-252/DPAK)"
- note added: "Door Switch"
- moved on the sheet: L1
